File: Schematics/DroneFlightController.sch (KiCad schematic (older format))
At the start: 0 parts

Commit message: add reference docs, rearrange schematics
Changed lines of the file:
@@
 $EndDescr
 $Sheet
-S 31700 4650 5050 4950
+S 18550 3650 5900 25750
 U 6125577D
 F0 "FMU_MCU_STM32H7" 50

Commit message: upnext, power
Other:
- note added: "CAN1 CONNECTORS"
- note added: "CAN2 CONNECTORS\n"
- note added: "ETHERNET CONNECTORS"
- note added: "FMU DEBUG CONNECTOR"
- note added: "I2C1 GPS1 CONNECTORS"
- note added: "I2C2 GPS2 CONNECTORS"
- note added: "I2C3 CONNECTORS"
- note added: "I2C4 BMP388 CONNECTORS"
- note added: "LEDS"
- note added: "MISCELLANEOUS"
- note added: "POWER MANAGEMENT"
- note added: "PWM CONNECTORS"
- note added: "RC CONNECTORS"
- note added: "SD1 CONNECTORS"
- note added: "SD2 CONNECTORS"
- note added: "SPI1 ICM20602 CONNECTORS"
- note added: "SPI2 ISM330 CONNECTORS"
- note added: "SPI3 BMI088 CONNECTORS\n"
- note added: "SPI4 BMM150 CONNECTORS"
- note added: "SPI5 FRAM CONNECTORS"
- note added: "SPI6 EXTERNAL CONNECTORS\n"
- note added: "UART4 CONNECTORS"
- note added: "USART2 TELEM3 CONNECTORS"
- note added: "USART5 TELEM2 CONNECTORS"
- note added: "USART7 TELEM1 CONNECTORS"
- note added: "USB C CONNECTORS"
